Commit message: stereo camera rpy modified

File: turtlebot4_description/urdf/sensors/oakd.urdf.xacro (robot description, xacro)
@@ -50,5 +50,5 @@
   </link>
   <joint name="${name}_rgb_camera_optical_joint" type="fixed">
-      <origin xyz="0 0 0" rpy="-${M_PI/2} 0.0 -${M_PI/2}"/>
+      <origin xyz="0 0 0" rpy="0 0.0 0"/>
       <parent link="${name}_rgb_camera_frame"/>
       <child link="${name}_rgb_camera_optical_frame"/>

Commit message: Restored code from a working commit

File: turtlebot4_description/urdf/sensors/oakd.urdf.xacro (robot description, xacro)
@@ -50,5 +50,5 @@
   </link>
   <joint name="${name}_rgb_camera_optical_joint" type="fixed">
-      <origin xyz="0 0 0" rpy="0 0.0 0"/>
+      <origin xyz="0 0 0" rpy="-${M_PI/2} 0.0 -${M_PI/2}"/>
       <parent link="${name}_rgb_camera_frame"/>
       <child link="${name}_rgb_camera_optical_frame"/>

File: turtlebot4_description/urdf/standard/turtlebot4.urdf.xacro (robot description, xacro)
@@ -93,5 +93,5 @@
   <xacro:rplidar name="rplidar" parent_link="shell_link" gazebo="$(arg gazebo)">
     <origin xyz="${rplidar_x_offset} ${rplidar_y_offset} ${rplidar_z_offset}"
-            rpy="0 0 0"/>
+            rpy="0 0 ${pi/2}"/>
   </xacro:rplidar>
   <xacro:camera_bracket name="oakd_camera_bracket">

Commit message: Added comment to explain why you did this change

File: turtlebot4_description/urdf/sensors/oakd.urdf.xacro (robot description, xacro)
@@ -50,4 +50,6 @@
   </link>
   <joint name="${name}_rgb_camera_optical_joint" type="fixed">
+      <!-- The following line has been modified to correctly align the point cloud in the simulation. If this configuration proves incompatible with the physical robot, you can implement conditional logic to select the appropriate setting based on the environment -->
+      <!-- <origin xyz="0 0 0" rpy="-${M_PI/2} 0.0 -${M_PI/2}"/> -->
       <origin xyz="0 0 0" rpy="0 0.0 0"/>
       <parent link="${name}_rgb_camera_frame"/>
